Commit message: add camera + nav2 docking

File: go1_gazebo/xacro/gazebo.xacro (robot description, xacro)
@@ -165,4 +165,27 @@
                 <topic>/${robot_name}/scan</topic>
                 <gz_frame_id>laser_frame</gz_frame_id>
+            </sensor>
+        </gazebo>
+        <gazebo reference="camera_face">
+            <!-- <material>Gazebo/Black</material> -->
+            <sensor name="camera" type="camera">
+                <pose> 0 0 0 0 0 0 </pose>
+                <visualize>true</visualize>
+                <update_rate>10</update_rate>
+                <camera>
+                    <camera_info_topic>/${robot_name}/color/camera_info</camera_info_topic>
+                    <horizontal_fov>1.089</horizontal_fov>
+                    <image>
+                        <format>R8G8B8</format>
+                        <width>640</width>
+                        <height>480</height>
+                    </image>
+                    <clip>
+                        <near>0.05</near>
+                        <far>8.0</far>
+                    </clip>
+                </camera>
+                <topic>/${robot_name}/color/image_raw</topic>
+                <gz_frame_id>camera_face</gz_frame_id>
             </sensor>
         </gazebo>

File: go1_gazebo/xacro/robot.xacro (robot description, xacro)
@@ -107,5 +107,5 @@
     <xacro:leg name="RL" mirror="1"  mirror_dae="True"   front_hind="-1" front_hind_dae="False" />
     <xacro:depthCamera camID="1" name="face">
-        <origin rpy="${PI} 0 0" xyz="0.2785 0.0125 0.0167"/>
+        <origin rpy="0 0 0" xyz="0.2785 0.0125 0.0167"/>
     </xacro:depthCamera>
     <xacro:depthCamera camID="2" name="chin">
