Commit message: go2 update

File: go2_gazebo/xacro/gazebo.xacro (robot description, xacro)
@@ -8,5 +8,5 @@
                 </ros>
                 <!-- <parameters>$(find go2_description)/config/gaz_ros2_ctl_use_sim.yaml</parameters> -->
-                <parameters>$(find go2_description)/config/ros_control/ros_control.yaml</parameters>
+                <parameters>$(find go2_gazebo)/config/ros_control/ros_control.yaml</parameters>
             </plugin>
         </gazebo>
@@ -88,4 +88,64 @@
             </joint>
         </ros2_control>
+        <gazebo reference="imu_link">
+            <!--<material>Gazebo/Black</material>-->
+            <gravity>false</gravity>
+            <sensor name="imu_sensor" type="imu">
+                <always_on>true</always_on>
+                <update_rate>100</update_rate>
+                <visualize>false</visualize>
+                <topic>/${robot_name}/imu_plugin/out</topic>
+                    <plugin filename="libgz-sim-imu-system.so" name="gz::sim::systems::Imu">
+                </plugin>
+                <pose>0 0 0 0 0 0</pose>
+                <gz_frame_id>imu_link</gz_frame_id> <!-- Добавьте этот тег для указания кадра -->
+            </sensor>
+        </gazebo>
+        <gazebo reference="laser_frame">
+            <!--<material>Gazebo/Black</material>-->
+            <sensor name="laser" type="gpu_lidar">
+                <pose> 0 0 0 0 0 0 </pose>
+                <visualize>false</visualize>
+                <update_rate>10</update_rate>
+                <lidar>
+                    <scan>
+                        <horizontal>
+                            <samples>360</samples>
+                            <min_angle>-3.14</min_angle>
+                            <max_angle>3.14</max_angle>
+                        </horizontal>
+                    </scan>
+                    <range>
+                        <min>0.3</min>
+                        <max>12</max>
+                    </range>
+                </lidar>
+                <topic>/${robot_name}/scan</topic>
+                <gz_frame_id>laser_frame</gz_frame_id>
+            </sensor>
+        </gazebo>
+        <gazebo reference="camera_face">
+            <!-- <material>Gazebo/Black</material> -->
+            <sensor name="camera" type="camera">
+                <pose> 0 0 0 0 0 0 </pose>
+                <visualize>true</visualize>
+                <update_rate>10</update_rate>
+                <camera>
+                    <camera_info_topic>/${robot_name}/color/camera_info</camera_info_topic>
+                    <horizontal_fov>1.089</horizontal_fov>
+                    <image>
+                        <format>R8G8B8</format>
+                        <width>640</width>
+                        <height>480</height>
+                    </image>
+                    <clip>
+                        <near>0.05</near>
+                        <far>8.0</far>
+                    </clip>
+                </camera>
+                <topic>/${robot_name}/color/image_raw</topic>
+                <gz_frame_id>camera_face</gz_frame_id>
+            </sensor>
+        </gazebo>
         <gazebo reference="trunk">
             <mu1>0.2</mu1>

File: go2_gazebo/xacro/laser.xacro (robot description, xacro)
@@ -17,5 +17,5 @@
         <origin rpy="0 0 0" xyz="0 0 0"/>
         <geometry>
-            <mesh filename="file://$(find go2_description)/meshes/hokuyo.dae"/>
+            <mesh filename="file://$(find go2_gazebo)/meshes/hokuyo.dae"/>
         </geometry>
         </visual>

File: go2_gazebo/xacro/leg.xacro (robot description, xacro)
@@ -1,5 +1,5 @@
 <?xml version="1.0"?>
 <robot xmlns:xacro="http://www.ros.org/wiki/xacro">
-    <!-- <xacro:include filename="$(find go2_description)/xacro/transmission.xacro"/> -->
+    <!-- <xacro:include filename="$(find go2_gazebo)/xacro/transmission.xacro"/> -->
     <xacro:macro name="leg" params="name mirror mirror_dae front_hind front_hind_dae">
         <joint name="${name}_hip_joint" type="revolute">
@@ -42,5 +42,5 @@
                 </xacro:if>
                 <geometry>
-                    <mesh filename="file://$(find go2_description)/meshes/hip.dae" scale="1 1 1"/>
+                    <mesh filename="file://$(find go2_gazebo)/meshes/hip.dae" scale="1 1 1"/>
                 </geometry>
                 <!-- <material name="orange"/> -->
@@ -74,8 +74,8 @@
                 <geometry>
                     <xacro:if value="${mirror_dae == True}">
-                        <mesh filename="file://$(find go2_description)/meshes/thigh.dae" scale="1 1 1"/>
+                        <mesh filename="file://$(find go2_gazebo)/meshes/thigh.dae" scale="1 1 1"/>
                     </xacro:if>
                     <xacro:if value="${mirror_dae == False}">
-                        <mesh filename="file://$(find go2_description)/meshes/thigh_mirror.dae" scale="1 1 1"/>
+                        <mesh filename="file://$(find go2_gazebo)/meshes/thigh_mirror.dae" scale="1 1 1"/>
                     </xacro:if>
                 </geometry>
@@ -109,5 +109,5 @@
                 <origin rpy="0 0 0" xyz="0 0 0"/>
                 <geometry>
-                    <mesh filename="file://$(find go2_description)/meshes/calf.dae" scale="1 1 1"/>
+                    <mesh filename="file://$(find go2_gazebo)/meshes/calf.dae" scale="1 1 1"/>
                 </geometry>
                 <!-- <material name="orange"/> -->

File: go2_gazebo/xacro/robot.xacro (robot description, xacro)
@@ -2,9 +2,9 @@
 <robot name="robot" xmlns:xacro="http://www.ros.org/wiki/xacro">
     <xacro:arg name="DEBUG" default="false"/>
-    <xacro:include filename="$(find go2_description)/xacro/const.xacro"/>
-    <xacro:include filename="$(find go2_description)/xacro/materials.xacro"/>
-    <xacro:include filename="$(find go2_description)/xacro/leg.xacro"/>
-    <!-- <xacro:include filename="$(find go2_description)/xacro/stairs.xacro"/> -->
-    <xacro:include filename="$(find go2_description)/xacro/gazebo.xacro"/>
+    <xacro:include filename="$(find go2_gazebo)/xacro/const.xacro"/>
+    <xacro:include filename="$(find go2_gazebo)/xacro/materials.xacro"/>
+    <xacro:include filename="$(find go2_gazebo)/xacro/leg.xacro"/>
+    <!-- <xacro:include filename="$(find go2_gazebo)/xacro/stairs.xacro"/> -->
+    <xacro:include filename="$(find go2_gazebo)/xacro/gazebo.xacro"/>
     <!-- <xacro:include filename="$(find go2_gazebo)/launch/stairs.urdf.xacro"/> -->
     <xacro:robot_gazebo_sensors robot_name="$(arg robot_name)"/>
@@ -38,5 +38,5 @@
             <origin rpy="0 0 0" xyz="0 0 0"/>
             <geometry>
-                <mesh filename="file://$(find go2_description)/meshes/trunk.dae" scale="1 1 1"/>
+                <mesh filename="file://$(find go2_gazebo)/meshes/trunk.dae" scale="1 1 1"/>
             </geometry>
             <!-- <material name="orange"/> -->
@@ -56,4 +56,54 @@
                 izz="${trunk_izz}"/>
         </inertial>
+    </link>
+    <joint name='laser_scan' type='fixed'>
+        <parent link="base_link"/>,
+        <child link="laser_frame"/>
+        <origin xyz="0.22 0.0 0.095" rpy="0 0 0" />
+    </joint>
+    <link name="laser_frame">
+        <inertial>
+            <mass value="0.001"/>
+            <origin rpy="0 0 0" xyz="0 0 0"/>
+            <inertia ixx="0.0001" ixy="0" ixz="0" iyy="0.0001" iyz="0" izz="0.0001"/>
+        </inertial>
+        <visual>
+            <origin rpy="0 0 0" xyz="0 0 0"/>
+            <geometry>
+                <cylinder length="0.01" radius="0.018" />
+            </geometry>
+            <!-- <material name="red"/> -->
+        </visual>
+        <collision>
+            <origin rpy="0 0 0" xyz="0 0 0"/>
+            <geometry>
+                <cylinder length="0.01" radius="0.018" />
+            </geometry>
+        </collision>
+    </link>
+    <joint name="imu_joint" type="fixed">
+        <parent link="base_link"/>
+        <child link="imu_link"/>
+        <origin rpy="0 0 0" xyz="0 0 0"/>
+    </joint>
+    <link name="imu_link">
+        <inertial>
+            <mass value="0.001"/>
+            <origin rpy="0 0 0" xyz="0 0 0"/>
+            <inertia ixx="0.0001" ixy="0" ixz="0" iyy="0.0001" iyz="0" izz="0.0001"/>
+        </inertial>
+        <visual>
+            <origin rpy="0 0 0" xyz="0 0 0"/>
+            <geometry>
+                <box size="0.001 0.001 0.001"/>
+            </geometry>
+            <!-- <material name="red"/> -->
+        </visual>
+        <collision>
+            <origin rpy="0 0 0" xyz="0 0 0"/>
+            <geometry>
+                <box size=".001 .001 .001"/>
+            </geometry>
+        </collision>
     </link>
     <!-- <joint name="imu_joint" type="fixed">

File: go2_gazebo/xacro/robot_VLP.xacro (robot description, xacro)
@@ -2,9 +2,9 @@
 <robot name="go2" xmlns:xacro="http://www.ros.org/wiki/xacro">
     <xacro:arg name="DEBUG" default="false"/>
-    <xacro:include filename="$(find go2_description)/xacro/const.xacro"/>
-    <xacro:include filename="$(find go2_description)/xacro/materials.xacro"/>
-    <xacro:include filename="$(find go2_description)/xacro/leg.xacro"/>
-    <!-- <xacro:include filename="$(find go2_description)/xacro/stairs.xacro"/> -->
-    <xacro:include filename="$(find go2_description)/xacro/gazebo.xacro"/>
+    <xacro:include filename="$(find go2_gazebo)/xacro/const.xacro"/>
+    <xacro:include filename="$(find go2_gazebo)/xacro/materials.xacro"/>
+    <xacro:include filename="$(find go2_gazebo)/xacro/leg.xacro"/>
+    <!-- <xacro:include filename="$(find go2_gazebo)/xacro/stairs.xacro"/> -->
+    <xacro:include filename="$(find go2_gazebo)/xacro/gazebo.xacro"/>
     <!-- <xacro:include filename="$(find go2_gazebo)/launch/stairs.urdf.xacro"/> -->
     <!-- <xacro:stairs stairs="15" xpos="0" ypos="0" zpos="0" /> -->
@@ -37,5 +37,5 @@
             <origin rpy="0 0 0" xyz="0 0 0"/>
             <geometry>
-                <mesh filename="file://$(find go2_description)/meshes/trunk.dae" scale="1 1 1"/>
+                <mesh filename="file://$(find go2_gazebo)/meshes/trunk.dae" scale="1 1 1"/>
             </geometry>
             <!-- <material name="orange"/> -->
@@ -110,5 +110,5 @@
     <xacro:leg name="rh" mirror="-1" mirror_dae="False"  front_hind="-1" front_hind_dae="False" />
     <xacro:leg name="lh" mirror="1"  mirror_dae="True"   front_hind="-1" front_hind_dae="False" />
-    <xacro:include filename="$(find go2_description)/xacro/velodyne.xacro"/>
-    <!-- <xacro:include filename="$(find go2_description)/xacro/laser.xacro"/> -->
+    <xacro:include filename="$(find go2_gazebo)/xacro/velodyne.xacro"/>
+    <!-- <xacro:include filename="$(find go2_gazebo)/xacro/laser.xacro"/> -->
 </robot>
