Commit message: gazebo classic

File: go1_description/xacro/gazebo.xacro (robot description, xacro)
@@ -361,6 +361,5 @@
         <kd  value="1.0"/>
     </gazebo>
-    <gazebo reference="imu_link">
-        <!--<material>Gazebo/Black</material>-->
+    <!-- <gazebo reference="imu_link">
         <gravity>false</gravity>
         <sensor name="imu_sensor" type="imu">
@@ -372,9 +371,8 @@
             </plugin>
             <pose>0 0 0 0 0 0</pose>
-            <gz_frame_id>imu_link</gz_frame_id> <!-- Добавьте этот тег для указания кадра -->
-        </sensor>
-    </gazebo>
-    <gazebo reference="laser_frame">
-        <!--<material>Gazebo/Black</material>-->
+            <gz_frame_id>imu_link</gz_frame_id>
+        </sensor>
+    </gazebo> -->
+    <!-- <gazebo reference="laser_frame">
         <sensor name="laser" type="gpu_lidar">
             <pose> 0 0 0 0 0 0 </pose>
@@ -397,6 +395,6 @@
             <gz_frame_id>laser_frame</gz_frame_id>
         </sensor>
-    </gazebo>
-    <gazebo>
+    </gazebo> -->
+    <!-- <gazebo>
         <plugin filename="ign_ros2_control-system" name="ign_ros2_control::IgnitionROS2ControlPlugin">
             <parameters>$(find go1_description)/config/gaz_ros2_ctl_use_sim.yaml</parameters>
@@ -480,4 +478,4 @@
         <state_interface name="effort"/>
         </joint>
-    </ros2_control>
+    </ros2_control> -->
 </robot>

Commit message: add namespace + nav2

File: go1_description/xacro/gazebo.xacro (robot description, xacro)
@@ -1,103 +1,312 @@
 <?xml version="1.0"?>
 <robot xmlns:xacro="http://www.ros.org/wiki/xacro" >
-    <!-- ros_control plugin -->
-    <!-- <gazebo>
-        <plugin name="gazebo_ros_control" filename="libgazebo_ros_control.so">
-            <robotNamespace>/go1_gazebo</robotNamespace>
-            <robotSimType>gazebo_ros_control/DefaultRobotHWSim</robotSimType>
-        </plugin>
-    </gazebo> -->
-    <!-- Show the trajectory of trunk center. -->
-    <!-- <gazebo>
-        <plugin name="3dplot" filename="libLinkPlot3DPlugin.so">
-            <frequency>10</frequency>
-            <plot>
-                <link>base</link>
+    <xacro:macro  name="robot_gazebo_sensors" params="robot_name">
+        <gazebo reference="base">
+            <!-- <material>Gazebo/Green</material> -->
+            <turnGravityOff>false</turnGravityOff>
+        </gazebo>
+        <gazebo reference="trunk">
+            <mu1>0.2</mu1>
+            <mu2>0.2</mu2>
+            <kp  value="1000000.0"/>
+            <kd  value="1.0"/>
+        </gazebo>
+        <gazebo reference="stick_link">
+            <mu1>0.2</mu1>
+            <mu2>0.2</mu2>
+            <material>Gazebo/White</material>
+        </gazebo>
+        <gazebo reference="imu_link">
+            <mu1>0.2</mu1>
+            <mu2>0.2</mu2>
+            <!-- <material>Gazebo/Red</material> -->
+        </gazebo>
+        <!-- FL leg -->
+        <gazebo reference="FL_hip">
+            <mu1>0.2</mu1>
+            <mu2>0.2</mu2>
+            <!--<material>Gazebo/DarkGrey</material>-->
+        </gazebo>
+        <gazebo reference="FL_thigh">
+            <mu1>0.2</mu1>
+            <mu2>0.2</mu2>
+            <self_collide>1</self_collide>
+            <!--<material>Gazebo/DarkGrey</material>-->
+            <kp  value="1000000.0"/>
+            <kd  value="1.0"/>
+        </gazebo>
+        <gazebo reference="FL_calf">
+            <mu1>0.2</mu1>
+            <mu2>0.2</mu2>
+            <self_collide>1</self_collide>
+        </gazebo>
+        <gazebo reference="FL_foot">
+            <mu1>0.6</mu1>
+            <mu2>0.6</mu2>
+            <self_collide>1</self_collide>
+            <!--<material>Gazebo/DarkGrey</material>-->
+            <kp  value="1000000.0"/>
+            <kd  value="1.0"/>
+        </gazebo>
+        <!-- FR leg -->
+        <gazebo reference="FR_hip">
+            <mu1>0.2</mu1>
+            <mu2>0.2</mu2>
+            <!--<material>Gazebo/DarkGrey</material>-->
+        </gazebo>
+        <gazebo reference="FR_thigh">
+            <mu1>0.2</mu1>
+            <mu2>0.2</mu2>
+            <self_collide>1</self_collide>
+            <!--<material>Gazebo/DarkGrey</material>-->
+            <kp  value="1000000.0"/>
+            <kd  value="1.0"/>
+        </gazebo>
+        <gazebo reference="FR_calf">
+            <mu1>0.2</mu1>
+            <mu2>0.2</mu2>
+            <self_collide>1</self_collide>
+        </gazebo>
+        <gazebo reference="FR_foot">
+            <mu1>0.6</mu1>
+            <mu2>0.6</mu2>
+            <self_collide>1</self_collide>
+            <!--<material>Gazebo/DarkGrey</material>-->
+            <kp  value="1000000.0"/>
+            <kd  value="1.0"/>
+        </gazebo>
+        <!-- RL leg -->
+        <gazebo reference="RL_hip">
+            <mu1>0.2</mu1>
+            <mu2>0.2</mu2>
+            <!--<material>Gazebo/DarkGrey</material>-->
+        </gazebo>
+        <gazebo reference="RL_thigh">
+            <mu1>0.2</mu1>
+            <mu2>0.2</mu2>
+            <self_collide>1</self_collide>
+            <!--<material>Gazebo/DarkGrey</material>-->
+            <kp  value="1000000.0"/>
+            <kd  value="1.0"/>
+        </gazebo>
+        <gazebo reference="RL_calf">
+            <mu1>0.2</mu1>
+            <mu2>0.2</mu2>
+            <self_collide>1</self_collide>
+        </gazebo>
+        <gazebo reference="RL_foot">
+            <mu1>0.6</mu1>
+            <mu2>0.6</mu2>
+            <self_collide>1</self_collide>
+            <!--<material>Gazebo/DarkGrey</material>-->
+            <kp  value="1000000.0"/>
+            <kd  value="1.0"/>
+        </gazebo>
+        <!-- RR leg -->
+        <gazebo reference="RR_hip">
+            <mu1>0.2</mu1>
+            <mu2>0.2</mu2>
+            <!--<material>Gazebo/DarkGrey</material>-->
+        </gazebo>
+        <gazebo reference="RR_thigh">
+            <mu1>0.2</mu1>
+            <mu2>0.2</mu2>
+            <self_collide>1</self_collide>
+            <!--<material>Gazebo/DarkGrey</material>-->
+            <kp  value="1000000.0"/>
+            <kd  value="1.0"/>
+        </gazebo>
+        <gazebo reference="RR_calf">
+            <mu1>0.2</mu1>
+            <mu2>0.2</mu2>
+            <self_collide>1</self_collide>
+        </gazebo>
+        <gazebo reference="RR_foot">
+            <mu1>0.6</mu1>
+            <mu2>0.6</mu2>
+            <self_collide>1</self_collide>
+            <!--<material>Gazebo/DarkGrey</material>-->
+            <kp  value="1000000.0"/>
+            <kd  value="1.0"/>
+        </gazebo>
+        <gazebo reference="imu_link">
+            <!--<material>Gazebo/Black</material>-->
+            <gravity>false</gravity>
+            <sensor name="imu_sensor" type="imu">
+                <always_on>true</always_on>
+                <update_rate>100</update_rate>
+                <visualize>false</visualize>
+                <topic>${robot_name}/imu_plugin/out</topic>
+                    <plugin filename="libgz-sim-imu-system.so" name="gz::sim::systems::Imu">
+                </plugin>
                 <pose>0 0 0 0 0 0</pose>
-                <material>Gazebo/Yellow</material>
-            </plot>
-        </plugin>
-    </gazebo> -->
-    <!-- Show the trajectory of foot. You can add another trajectory about another foot. -->
-    <!-- <gazebo>
-        <plugin name="3dplot" filename="libLinkPlot3DPlugin.so">
-            <frequency>100</frequency>
-            <plot>
-                <link>FL_foot</link>
+                <gz_frame_id>imu_link</gz_frame_id> <!-- Добавьте этот тег для указания кадра -->
+            </sensor>
+        </gazebo>
+        <gazebo reference="laser_frame">
+            <!--<material>Gazebo/Black</material>-->
+            <sensor name="laser" type="gpu_lidar">
+                <pose> 0 0 0 0 0 0 </pose>
+                <visualize>false</visualize>
+                <update_rate>10</update_rate>
+                <lidar>
+                    <scan>
+                        <horizontal>
+                            <samples>360</samples>
+                            <min_angle>-3.14</min_angle>
+                            <max_angle>3.14</max_angle>
+                        </horizontal>
+                    </scan>
+                    <range>
+                        <min>0.3</min>
+                        <max>12</max>
+                    </range>
+                </lidar>
+                <topic>${robot_name}/scan</topic>
+                <gz_frame_id>laser_frame</gz_frame_id>
+            </sensor>
+        </gazebo>
+        <gazebo>
+            <plugin filename="ign_ros2_control-system" name="ign_ros2_control::IgnitionROS2ControlPlugin">
+                <ros>
+                    <namespace>/${robot_name}</namespace>
+                </ros>
+                <parameters>$(find go1_description)/config/gaz_ros2_ctl_use_sim.yaml</parameters>
+                <parameters>$(find go1_description)/config/robot_control.yaml</parameters>
+            </plugin>
+        </gazebo>
+        <ros2_control name="${robot_name}_IgnitionSystem" type="system">
+            <hardware>
+                <plugin>ign_ros2_control/IgnitionSystem</plugin>
+            </hardware>
+            <joint name="FL_hip_joint">
+            <command_interface name="position"/>
+            <state_interface name="position"/>
+            <state_interface name="velocity"/>
+            <state_interface name="effort"/>
+            </joint>
+            <joint name="FL_thigh_joint">
+            <command_interface name="position"/>
+            <state_interface name="position"/>
+            <state_interface name="velocity"/>
+            <state_interface name="effort"/>
+            </joint>
+            <joint name="FL_calf_joint">
+            <command_interface name="position"/>
+            <state_interface name="position"/>
+            <state_interface name="velocity"/>
+            <state_interface name="effort"/>
+            </joint>
+            <joint name="FR_hip_joint">
+            <command_interface name="position"/>
+            <state_interface name="position"/>
+            <state_interface name="velocity"/>
+            <state_interface name="effort"/>
+            </joint>
+            <joint name="FR_thigh_joint">
+            <command_interface name="position"/>
+            <state_interface name="position"/>
+            <state_interface name="velocity"/>
+            <state_interface name="effort"/>
+            </joint>
+            <joint name="FR_calf_joint">
+            <command_interface name="position"/>
+            <state_interface name="position"/>
+            <state_interface name="velocity"/>
+            <state_interface name="effort"/>
+            </joint>
+            <joint name="RL_hip_joint">
+            <command_interface name="position"/>
+            <state_interface name="position"/>
+            <state_interface name="velocity"/>
+            <state_interface name="effort"/>
+            </joint>
+            <joint name="RL_thigh_joint">
+            <command_interface name="position"/>
+            <state_interface name="position"/>
+            <state_interface name="velocity"/>
+            <state_interface name="effort"/>
+            </joint>
+            <joint name="RL_calf_joint">
+            <command_interface name="position"/>
+            <state_interface name="position"/>
+            <state_interface name="velocity"/>
+            <state_interface name="effort"/>
+            </joint>
+            <joint name="RR_hip_joint">
+            <command_interface name="position"/>
+            <state_interface name="position"/>
+            <state_interface name="velocity"/>
+            <state_interface name="effort"/>
+            </joint>
+            <joint name="RR_thigh_joint">
+            <command_interface name="position"/>
+            <state_interface name="position"/>
+            <state_interface name="velocity"/>
+            <state_interface name="effort"/>
+            </joint>
+            <joint name="RR_calf_joint">
+            <command_interface name="position"/>
+            <state_interface name="position"/>
+            <state_interface name="velocity"/>
+            <state_interface name="effort"/>
+            </joint>
+        </ros2_control>
+                <!-- ros_control plugin -->
+        <!-- <gazebo>
+            <plugin name="gazebo_ros_control" filename="libgazebo_ros_control.so">
+                <robotNamespace>/go1_gazebo</robotNamespace>
+                <robotSimType>gazebo_ros_control/DefaultRobotHWSim</robotSimType>
+            </plugin>
+        </gazebo> -->
+        <!-- Show the trajectory of trunk center. -->
+        <!-- <gazebo>
+            <plugin name="3dplot" filename="libLinkPlot3DPlugin.so">
+                <frequency>10</frequency>
+                <plot>
+                    <link>base</link>
+                    <pose>0 0 0 0 0 0</pose>
+                    <material>Gazebo/Yellow</material>
+                </plot>
+            </plugin>
+        </gazebo> -->
+        <!-- Show the trajectory of foot. You can add another trajectory about another foot. -->
+        <!-- <gazebo>
+            <plugin name="3dplot" filename="libLinkPlot3DPlugin.so">
+                <frequency>100</frequency>
+                <plot>
+                    <link>FL_foot</link>
+                    <pose>0 0 0 0 0 0</pose>
+                    <material>Gazebo/Green</material>
+                </plot>
+            </plugin>
+        </gazebo> -->
+        <!-- <gazebo>
+            <plugin filename="libgazebo_ros_force.so" name="gazebo_ros_force">
+                <bodyName>trunk</bodyName>
+                <topicName>/apply_force/trunk</topicName>
+            </plugin>
+        </gazebo> -->
+        <!-- <gazebo reference="imu_link">
+            <gravity>true</gravity>
+            <sensor name="imu_sensor" type="imu">
+                <always_on>true</always_on>
+                <update_rate>1000</update_rate>
+                <visualize>true</visualize>
+                <topic>__default_topic__</topic>
+                <plugin filename="libgazebo_ros_imu_sensor.so" name="imu_plugin">
+                    <topicName>trunk_imu</topicName>
+                    <bodyName>imu_link</bodyName>
+                    <updateRateHZ>1000.0</updateRateHZ>
+                    <gaussianNoise>0.0</gaussianNoise>
+                    <xyzOffset>0 0 0</xyzOffset>
+                    <rpyOffset>0 0 0</rpyOffset>
+                    <frameName>imu_link</frameName>
+                </plugin>
                 <pose>0 0 0 0 0 0</pose>
-                <material>Gazebo/Green</material>
-            </plot>
-        </plugin>
-    </gazebo> -->
-    <!-- <gazebo>
-        <plugin filename="libgazebo_ros_force.so" name="gazebo_ros_force">
-            <bodyName>trunk</bodyName>
-            <topicName>/apply_force/trunk</topicName>
-        </plugin>
-    </gazebo> -->
-    <!-- <gazebo reference="imu_link">
-        <gravity>true</gravity>
-        <sensor name="imu_sensor" type="imu">
-            <always_on>true</always_on>
-            <update_rate>1000</update_rate>
-            <visualize>true</visualize>
-            <topic>__default_topic__</topic>
-            <plugin filename="libgazebo_ros_imu_sensor.so" name="imu_plugin">
-                <topicName>trunk_imu</topicName>
-                <bodyName>imu_link</bodyName>
-                <updateRateHZ>1000.0</updateRateHZ>
-                <gaussianNoise>0.0</gaussianNoise>
-                <xyzOffset>0 0 0</xyzOffset>
-                <rpyOffset>0 0 0</rpyOffset>
-                <frameName>imu_link</frameName>
-            </plugin>
-            <pose>0 0 0 0 0 0</pose>
-        </sensor>
-    </gazebo> -->
-    <!-- Depth camera -->
-    <!-- <gazebo>
-        <plugin name="camera_plugin" filename="libgazebo_ros_openni_kinect.so">
-            <baseline>0.025</baseline>
-            <always_on>true</always_on>
-            <updateRate>0.0</updateRate>
-            <cameraName>unitree_camera_left</cameraName>
-            <frameName>depthCamera_link_left</frameName>
-            <imageTopicName>rgb/imageRaw_left</imageTopicName>
-            <depthImageTopicName>depth/imageRaw_left</depthImageTopicName>
-            <pointCloudTopicName>depth/points_left</pointCloudTopicName>
-            <cameraInfoTopicName>rgb/cameraInfo_left</cameraInfoTopicName>
-            <depthImageCameraInfoTopicName>depth/cameraInfo_left</depthImageCameraInfoTopicName>
-            <pointCloudCutoff>0.1</pointCloudCutoff>
-            <pointCloudCutoffMax>1.5</pointCloudCutoffMax>
-            <distortionK1>0.0</distortionK1>
-            <distortionK2>0.0</distortionK2>
-            <distortionK3>0.0</distortionK3>
-            <distortionT1>0.0</distortionT1>
-            <distortionT2>0.0</distortionT2>
-            <CxPrime>0.0</CxPrime>
-            <Cx>0.0045</Cx>
-            <Cy>0.0039</Cy>
-            <focalLength>0.004</focalLength>
-            <hackBaseline>0.0</hackBaseline>
-        </plugin>
-    </gazebo> -->
-    <!-- <gazebo reference="depthCamera_link_left">
-        <sensor name="unitree_camera_left" type="depth_camera">
-            <update_rate>16</update_rate>
-            <always_on>true</always_on>
-            <visualize>true</visualize>
-            <camera>
-                <horizontal_fov>2.094</horizontal_fov>
-                <image>
-                    <width>928</width>
-                    <height>800</height>
-                    <format>R8G8B8</format>
-                </image>
-                <depth_camera></depth_camera>
-                <clip>
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
File: go1_description/xacro/robot.xacro (robot description, xacro)
@@ -14,16 +14,5 @@
     <xacro:include filename="$(find go1_description)/xacro/ultraSound.xacro"/> -->
     <!-- <xacro:include filename="$(find go1_gazebo)/launch/stairs.urdf.xacro"/> -->
-    <!-- <xacro:stairs stairs="15" xpos="0" ypos="0" zpos="0" /> -->
-    <!-- Rotor related joint and link is only for demonstrate location. -->
-    <!-- Actually, the rotor will rotate and the joint is not fixed. Reduction ratio should be considered. -->
-    <!-- Debug mode will hung up the robot, use "true" or "false" to switch it. -->
-    <!-- <xacro:if value="$(arg DEBUG)">
-        <link name="world"/>
-        <joint name="base_static_joint" type="fixed">
-            <origin rpy="0 0 0" xyz="0 0 0"/>
-            <parent link="world"/>
-            <child link="base"/>
-        </joint>
-    </xacro:if>  -->
+    <xacro:robot_gazebo_sensors robot_name="$(arg robot_name)"/>
     <joint name='laser_scan' type='fixed'>
         <parent link="base"/>,
@@ -53,34 +42,4 @@
     <link name="base">
     </link>
-    <!-- <xacro:if value="$(arg use_nav2_links)">
-        <link name="base_link" >
-        </link>
-        <joint name="base_link_to_base" type="fixed">
-            <origin rpy="0 0 0" xyz="0 0 0"/>
-            <parent link="base_link"/>
-            <child link="base"/>
-        </joint>
-        <link name="height_measurement" />
-        <joint name="base_link_to_height" type="fixed">
-            <origin rpy="0 0 0" xyz="0 0 -0.015"/>
-            <parent link="base_link"/>
-            <child link="height_measurement"/>
-        </joint>
-        <link name="base_footprint" >
-        </link>
-        <joint name="height_to_footprint" type="prismatic">
-                <parent link="height_measurement"/>
-                <child link="base_footprint"/>
-                <origin xyz = "0 0 0" rpy="0 0 0"/>
-                <axis xyz="0 0 -1" />
-                <limit effort="100000.0" lower="0.0" upper="1.0" velocity="100000.0"/>
-        </joint>
-        <link name="base_laser" />
-        <joint name="base_link_to_lidar" type="fixed">
-            <origin rpy="0 0 0" xyz="$(arg lidar_x_offset) $(arg lidar_y_offset) $(arg lidar_z_offset)"/>
-            <parent link="base_link"/>
-            <child link="base_laser"/>
-        </joint>
-    </xacro:if> -->
     <joint name="floating_base" type="fixed">
         <origin rpy="0 0 0" xyz="0 0 0"/>
