Commit message: odom with interface

File: go1_description/xacro/gazebo.xacro (robot description, xacro)
@@ -130,8 +130,8 @@
             <kd  value="1.0"/>
         </gazebo>
-        <gazebo reference="${robot_name}_imu_link">
+        <gazebo reference="imu_link">
             <!--<material>Gazebo/Black</material>-->
             <gravity>false</gravity>
-            <sensor name="${robot_name}_imu_sensor" type="imu">
+            <sensor name="imu_sensor" type="imu">
                 <always_on>true</always_on>
                 <update_rate>100</update_rate>
@@ -141,10 +141,10 @@
                 </plugin>
                 <pose>0 0 0 0 0 0</pose>
-                <gz_frame_id>${robot_name}_imu_link</gz_frame_id> <!-- Добавьте этот тег для указания кадра -->
-            </sensor>
-        </gazebo>
-        <gazebo reference="${robot_name}_laser_frame">
+                <gz_frame_id>imu_link</gz_frame_id> <!-- Добавьте этот тег для указания кадра -->
+            </sensor>
+        </gazebo>
+        <gazebo reference="laser_frame">
             <!--<material>Gazebo/Black</material>-->
-            <sensor name="${robot_name}_laser" type="gpu_lidar">
+            <sensor name="laser" type="gpu_lidar">
                 <pose> 0 0 0 0 0 0 </pose>
                 <visualize>false</visualize>
@@ -164,5 +164,5 @@
                 </lidar>
                 <topic>${robot_name}/scan</topic>
-                <gz_frame_id>${robot_name}_laser_frame</gz_frame_id>
+                <gz_frame_id>laser_frame</gz_frame_id>
             </sensor>
         </gazebo>
@@ -180,71 +180,71 @@
                 <plugin>ign_ros2_control/IgnitionSystem</plugin>
             </hardware>
-            <joint name="${robot_name}_FL_hip_joint">
-            <command_interface name="position"/>
-            <state_interface name="position"/>
-            <state_interface name="velocity"/>
-            <state_interface name="effort"/>
-            </joint>
-            <joint name="${robot_name}_FL_thigh_joint">
-            <command_interface name="position"/>
-            <state_interface name="position"/>
-            <state_interface name="velocity"/>
-            <state_interface name="effort"/>
-            </joint>
-            <joint name="${robot_name}_FL_calf_joint">
-            <command_interface name="position"/>
-            <state_interface name="position"/>
-            <state_interface name="velocity"/>
-            <state_interface name="effort"/>
-            </joint>
-            <joint name="${robot_name}_FR_hip_joint">
-            <command_interface name="position"/>
-            <state_interface name="position"/>
-            <state_interface name="velocity"/>
-            <state_interface name="effort"/>
-            </joint>
-            <joint name="${robot_name}_FR_thigh_joint">
-            <command_interface name="position"/>
-            <state_interface name="position"/>
-            <state_interface name="velocity"/>
-            <state_interface name="effort"/>
-            </joint>
-            <joint name="${robot_name}_FR_calf_joint">
-            <command_interface name="position"/>
-            <state_interface name="position"/>
-            <state_interface name="velocity"/>
-            <state_interface name="effort"/>
-            </joint>
-            <joint name="${robot_name}_RL_hip_joint">
-            <command_interface name="position"/>
-            <state_interface name="position"/>
-            <state_interface name="velocity"/>
-            <state_interface name="effort"/>
-            </joint>
-            <joint name="${robot_name}_RL_thigh_joint">
-            <command_interface name="position"/>
-            <state_interface name="position"/>
-            <state_interface name="velocity"/>
-            <state_interface name="effort"/>
-            </joint>
-            <joint name="${robot_name}_RL_calf_joint">
-            <command_interface name="position"/>
-            <state_interface name="position"/>
-            <state_interface name="velocity"/>
-            <state_interface name="effort"/>
-            </joint>
-            <joint name="${robot_name}_RR_hip_joint">
-            <command_interface name="position"/>
-            <state_interface name="position"/>
-            <state_interface name="velocity"/>
-            <state_interface name="effort"/>
-            </joint>
-            <joint name="${robot_name}_RR_thigh_joint">
-            <command_interface name="position"/>
-            <state_interface name="position"/>
-            <state_interface name="velocity"/>
-            <state_interface name="effort"/>
-            </joint>
-            <joint name="${robot_name}_RR_calf_joint">
+            <joint name="FL_hip_joint">
+            <command_interface name="position"/>
+            <state_interface name="position"/>
+            <state_interface name="velocity"/>
+            <state_interface name="effort"/>
+            </joint>
+            <joint name="FL_thigh_joint">
+            <command_interface name="position"/>
+            <state_interface name="position"/>
+            <state_interface name="velocity"/>
+            <state_interface name="effort"/>
+            </joint>
+            <joint name="FL_calf_joint">
+            <command_interface name="position"/>
+            <state_interface name="position"/>
+            <state_interface name="velocity"/>
+            <state_interface name="effort"/>
+            </joint>
+            <joint name="FR_hip_joint">
+            <command_interface name="position"/>
+            <state_interface name="position"/>
+            <state_interface name="velocity"/>
+            <state_interface name="effort"/>
+            </joint>
+            <joint name="FR_thigh_joint">
+            <command_interface name="position"/>
+            <state_interface name="position"/>
+            <state_interface name="velocity"/>
+            <state_interface name="effort"/>
+            </joint>
+            <joint name="FR_calf_joint">
+            <command_interface name="position"/>
+            <state_interface name="position"/>
+            <state_interface name="velocity"/>
+            <state_interface name="effort"/>
+            </joint>
+            <joint name="RL_hip_joint">
+            <command_interface name="position"/>
+            <state_interface name="position"/>
+            <state_interface name="velocity"/>
+            <state_interface name="effort"/>
+            </joint>
+            <joint name="RL_thigh_joint">
+            <command_interface name="position"/>
+            <state_interface name="position"/>
+            <state_interface name="velocity"/>
+            <state_interface name="effort"/>
+            </joint>
+            <joint name="RL_calf_joint">
+            <command_interface name="position"/>
+            <state_interface name="position"/>
+            <state_interface name="velocity"/>
+            <state_interface name="effort"/>
+            </joint>
+            <joint name="RR_hip_joint">
+            <command_interface name="position"/>
+            <state_interface name="position"/>
+            <state_interface name="velocity"/>
+            <state_interface name="effort"/>
+            </joint>
+            <joint name="RR_thigh_joint">
+            <command_interface name="position"/>
+            <state_interface name="position"/>
+            <state_interface name="velocity"/>
+            <state_interface name="effort"/>
+            </joint>
+            <joint name="RR_calf_joint">
             <command_interface name="position"/>
             <state_interface name="position"/>

File: go1_description/xacro/leg.xacro (robot description, xacro)
@@ -1,8 +1,7 @@
 <?xml version="1.0"?>
 <robot xmlns:xacro="http://www.ros.org/wiki/xacro">
-    <xacro:macro name="leg" params="robot_name name mirror mirror_dae front_hind front_hind_dae">
-        <!-- Сустав hip_joint с уникализированным именем -->
-        <joint name="${robot_name}_${name}_hip_joint" type="revolute">
-            <!-- Установка позиции и ориентации сустава в зависимости от параметров mirror_dae и front_hind_dae -->
+    <xacro:include filename="$(find go1_description)/xacro/transmission.xacro"/>
+    <xacro:macro name="leg" params="name mirror mirror_dae front_hind front_hind_dae">
+        <joint name="${name}_hip_joint" type="revolute">
             <xacro:if value="${(mirror_dae == False) and (front_hind_dae == True)}">
                 <origin rpy="0 0 0" xyz="${leg_offset_x} ${-leg_offset_y} 0"/>
@@ -17,9 +16,8 @@
                 <origin rpy="0 0 0" xyz="${-leg_offset_x} ${leg_offset_y} 0"/>
             </xacro:if>
-            <parent link="${robot_name}_trunk"/>
-            <child link="${robot_name}_${name}_hip"/>
+            <parent link="trunk"/>
+            <child link="${name}_hip"/>
             <axis xyz="1 0 0"/>
             <dynamics damping="${damping}" friction="${friction}"/>
-            <!-- Настройка ограничений для сустава в зависимости от mirror_dae -->
             <xacro:if value="${(mirror_dae == True)}">
                 <limit effort="${hip_torque_max}" velocity="${hip_velocity_max}" lower="${hip_position_min}" upper="${hip_position_max}"/>
@@ -29,6 +27,5 @@
             </xacro:if>
         </joint>
-        <!-- Сустав hip_rotor_joint с уникализированным именем -->
-        <joint name="${robot_name}_${name}_hip_rotor_joint" type="fixed">
+        <joint name="${name}_hip_rotor_joint" type="fixed">
             <xacro:if value="${(mirror_dae == False) and (front_hind_dae == True)}">
                 <origin rpy="0 0 0" xyz="${hip_rotor_offset_x} ${-hip_rotor_offset_y} 0"/>
@@ -43,9 +40,8 @@
                 <origin rpy="0 0 0" xyz="${-hip_rotor_offset_x} ${hip_rotor_offset_y} 0"/>
             </xacro:if>
-            <parent link="${robot_name}_trunk"/>
-            <child link="${robot_name}_${name}_hip_rotor"/>
-        </joint>
-        <!-- Ссылка hip с уникализированным именем -->
-        <link name="${robot_name}_${name}_hip">
+            <parent link="trunk"/>
+            <child link="${name}_hip_rotor"/>
+        </joint>
+        <link name="${name}_hip">
             <visual>
                 <xacro:if value="${(mirror_dae == True) and (front_hind_dae == True)}">
@@ -81,6 +77,5 @@
             </inertial>
         </link>
-        <!-- Ссылка hip_rotor с уникализированным именем -->
-        <link name="${robot_name}_${name}_hip_rotor">
+        <link name="${name}_hip_rotor">
             <visual>
                 <origin rpy="0 ${PI/2.0} 0" xyz="0 0 0"/>
@@ -105,21 +100,18 @@
             </inertial>
         </link>
-        <!-- Сустав thigh_joint с уникализированным именем -->
-        <joint name="${robot_name}_${name}_thigh_joint" type="revolute">
+        <joint name="${name}_thigh_joint" type="revolute">
             <origin rpy="0 0 0" xyz="0 ${thigh_offset*mirror} 0"/>
-            <parent link="${robot_name}_${name}_hip"/>
-            <child link="${robot_name}_${name}_thigh"/>
+            <parent link="${name}_hip"/>
+            <child link="${name}_thigh"/>
             <axis xyz="0 1 0"/>
             <dynamics damping="${damping}" friction="${friction}"/>
             <limit effort="${thigh_torque_max}" velocity="${thigh_velocity_max}" lower="${thigh_position_min}" upper="${thigh_position_max}"/>
         </joint>
-        <!-- Сустав thigh_rotor_joint с уникализированным именем -->
-        <joint name="${robot_name}_${name}_thigh_rotor_joint" type="fixed">
+        <joint name="${name}_thigh_rotor_joint" type="fixed">
             <origin rpy="0 0 0" xyz="${thigh_rotor_offset_x} ${thigh_rotor_offset_y*mirror} 0"/>
-            <parent link="${robot_name}_${name}_hip"/>
-            <child link="${robot_name}_${name}_thigh_rotor"/>
-        </joint>
-        <!-- Ссылка thigh с уникализированным именем -->
-        <link name="${robot_name}_${name}_thigh">
+            <parent link="${name}_hip"/>
+            <child link="${name}_thigh_rotor"/>
+        </joint>
+        <link name="${name}_thigh">
             <visual>
                 <origin rpy="0 0 0" xyz="0 0 0"/>
@@ -149,6 +141,5 @@
             </inertial>
         </link>
-        <!-- Ссылка thigh_rotor с уникализированным именем -->
-        <link name="${robot_name}_${name}_thigh_rotor">
+        <link name="${name}_thigh_rotor">
             <visual>
                 <origin rpy="${PI/2.0} 0 0" xyz="0 0 0"/>
@@ -173,21 +164,18 @@
             </inertial>
         </link>
-        <!-- Сустав calf_joint с уникализированным именем -->
-        <joint name="${robot_name}_${name}_calf_joint" type="revolute">
+        <joint name="${name}_calf_joint" type="revolute">
             <origin rpy="0 0 0" xyz="0 0 ${-thigh_length}"/>
-            <parent link="${robot_name}_${name}_thigh"/>
-            <child link="${robot_name}_${name}_calf"/>
+            <parent link="${name}_thigh"/>
+            <child link="${name}_calf"/>
             <axis xyz="0 1 0"/>
             <dynamics damping="${damping}" friction="${friction}"/>
             <limit effort="${calf_torque_max}" velocity="${calf_velocity_max}" lower="${calf_position_min}" upper="${calf_position_max}"/>
         </joint>
-        <!-- Сустав calf_rotor_joint с уникализированным именем -->
-        <joint name="${robot_name}_${name}_calf_rotor_joint" type="fixed">
+        <joint name="${name}_calf_rotor_joint" type="fixed">
             <origin rpy="0 0 0" xyz="${calf_rotor_offset_x} ${calf_rotor_offset_y*mirror} 0"/>
-            <parent link="${robot_name}_${name}_thigh"/>
-            <child link="${robot_name}_${name}_calf_rotor"/>
-        </joint>
-        <!-- Ссылка calf с уникализированным именем -->
-        <link name="${robot_name}_${name}_calf">
+            <parent link="${name}_thigh"/>
+            <child link="${name}_calf_rotor"/>
+        </joint>
+        <link name="${name}_calf">
             <visual>
                 <origin rpy="0 0 0" xyz="0 0 0"/>
@@ -212,6 +200,5 @@
             </inertial>
         </link>
-        <!-- Ссылка calf_rotor с уникализированным именем -->
-        <link name="${robot_name}_${name}_calf_rotor">
+        <link name="${name}_calf_rotor">
             <visual>
                 <origin rpy="${PI/2.0} 0 0" xyz="0 0 0"/>
@@ -236,16 +223,14 @@
             </inertial>
         </link>
-        <!-- Сустав foot_fixed с уникализированным именем -->
-        <joint name="${robot_name}_${name}_foot_fixed" type="fixed">
+        <joint name="${name}_foot_fixed" type="fixed">
             <origin rpy="0 0 0" xyz="0 0 ${-(calf_length)}"/>
-            <parent link="${robot_name}_${name}_calf"/>
-            <child link="${robot_name}_${name}_foot"/>
-        </joint>
-        <!-- Ссылка foot с уникализированным именем -->
-        <link name="${robot_name}_${name}_foot">
-            <visual>
-                <origin rpy="0 0 0" xyz="0 0 0"/>
-                <geometry>
-                    <sphere radius="${foot_radius - 0.01}"/>
+            <parent link="${name}_calf"/>
+            <child link="${name}_foot"/>
+        </joint>
+        <link name="${name}_foot">
+            <visual>
+                <origin rpy="0 0 0" xyz="0 0 0"/>
+                <geometry>
+                    <sphere radius="${foot_radius-0.01}"/>
                 </geometry>
                 <!-- <material name="orange"/> -->
@@ -260,11 +245,10 @@
                 <mass value="${foot_mass}"/>
                 <inertia
-                    ixx="${(2 * foot_mass) / 5.0 * (foot_radius * foot_radius)}" ixy="0.0" ixz="0.0"
-                    iyy="${(2 * foot_mass) / 5.0 * (foot_radius * foot_radius)}" iyz="0.0"
-                    izz="${(2 * foot_mass) / 5.0 * (foot_radius * foot_radius)}"/>
-            </inertial>
-        </link>
-        <!-- Передача уникализированного имени для transmission -->
-        <xacro:leg_transmission robot_name="${robot_name}" name="${name}"/>
+                    ixx="${(2*foot_mass)/5.0*(foot_radius*foot_radius)}" ixy="0.0" ixz="0.0"
+                    iyy="${(2*foot_mass)/5.0*(foot_radius*foot_radius)}" iyz="0.0"
+                    izz="${(2*foot_mass)/5.0*(foot_radius*foot_radius)}"/>
+            </inertial>
+        </link>
+        <xacro:leg_transmission name="${name}"/>
     </xacro:macro>
 </robot>
