Commit message: odom with interface

File: go1_description/xacro/robot.xacro (robot description, xacro)
@@ -1,7 +1,4 @@
 <?xml version="1.0"?>
-<!-- robot.xacro -->
-<robot name="$(arg robot_name)" xmlns:xacro="http://www.ros.org/wiki/xacro">
-    <!-- Определение аргументов -->
-    <!-- <xacro:arg name="robot_name" default="robot1"/> -->
+<robot name="robot" xmlns:xacro="http://www.ros.org/wiki/xacro">
     <xacro:arg name="DEBUG" default="false"/>
     <xacro:arg name="use_nav2_links" default="False"/>
@@ -9,24 +6,19 @@
     <xacro:arg name="lidar_y_offset" default="0.0"/>
     <xacro:arg name="lidar_z_offset" default="0.21"/>
-    <!-- Определение префикса для уникализации имен -->
-    <xacro:property name="prefix" value="$(arg robot_name)_"/>
-    <!-- Включение необходимых Xacro файлов -->
     <xacro:include filename="$(find go1_description)/xacro/const.xacro"/>
     <xacro:include filename="$(find go1_description)/xacro/materials.xacro"/>
+    <xacro:include filename="$(find go1_description)/xacro/leg.xacro"/>
+    <!-- <xacro:include filename="$(find go1_description)/xacro/stairs.xacro"/> -->
     <xacro:include filename="$(find go1_description)/xacro/gazebo.xacro"/>
-    <xacro:include filename="$(find go1_description)/xacro/leg.xacro"/>
-    <xacro:include filename="$(find go1_description)/xacro/transmission.xacro"/>
-    <!-- Включение сенсоров -->
+    <!-- <xacro:include filename="$(find go1_description)/xacro/depthCamera.xacro"/>
+    <xacro:include filename="$(find go1_description)/xacro/ultraSound.xacro"/> -->
+    <!-- <xacro:include filename="$(find go1_gazebo)/launch/stairs.urdf.xacro"/> -->
     <xacro:robot_gazebo_sensors robot_name="$(arg robot_name)"/>
-    <!-- Вызов макроса legs для создания всех ног -->
-    <!-- <xacro:robot_gazebo_legs robot_name="$(arg robot_name)"/> -->
-    <!-- Сустав для лазера с уникализированным именем -->
-    <joint name='${prefix}laser_scan' type='fixed'>
-        <parent link="${prefix}base"/>
-        <child link="${prefix}laser_frame"/>
+    <joint name='laser_scan' type='fixed'>
+        <parent link="base"/>,
+        <child link="laser_frame"/>
         <origin xyz="0.263 0.0 0.077" rpy="0 0 0" />
     </joint>
-    <!-- Ссылка для лазера с уникализированным именем -->
-    <link name="${prefix}laser_frame">
+    <link name="laser_frame">
         <inertial>
             <mass value="0.001"/>
@@ -48,24 +40,19 @@
         </collision>
     </link>
-    <!-- Базовая ссылка с уникализированным именем -->
-    <link name="${prefix}base">
+    <link name="base">
     </link>
-    <!-- Сустав для плавающей базы с уникализированным именем -->
-    <joint name="${prefix}floating_base" type="fixed">
+    <joint name="floating_base" type="fixed">
         <origin rpy="0 0 0" xyz="0 0 0"/>
-        <parent link="${prefix}base"/>
-        <child link="${prefix}trunk"/>
+        <parent link="base"/>
+        <child link="trunk"/>
     </joint>
-    <!-- Ссылка для базового фундамента с уникализированным именем -->
-    <link name="${prefix}base_footprint">
+    <link name="base_footprint" >
     </link>
-    <!-- Сустав для базового фундамента с уникализированным именем -->
-    <joint name="${prefix}base_footprint_joint" type="fixed">
-        <parent link="${prefix}base"/>
-        <child link="${prefix}base_footprint"/>
+    <joint name="base_footprint_joint" type="fixed">
+        <parent link="base"/>
+        <child link="base_footprint"/>
         <origin xyz="0 0 0" rpy="0 0 0"/>
     </joint>
-    <!-- Ссылка для трака с уникализированным именем -->
-    <link name="${prefix}trunk">
+    <link name="trunk">
         <visual>
             <origin rpy="0 0 0" xyz="0 0 0"/>
@@ -90,12 +77,10 @@
         </inertial>
     </link>
-    <!-- Сустав для IMU с уникализированным именем -->
-    <joint name="${prefix}imu_joint" type="fixed">
-        <parent link="${prefix}base"/>
-        <child link="${prefix}imu_link"/>
+    <joint name="imu_joint" type="fixed">
+        <parent link="base"/>
+        <child link="imu_link"/>
         <origin rpy="0 0 0" xyz="0 0 0"/>
     </joint>
-    <!-- Ссылка для IMU с уникализированным именем -->
-    <link name="${prefix}imu_link">
+    <link name="imu_link">
         <inertial>
             <mass value="0.001"/>
@@ -117,49 +102,45 @@
         </collision>
     </link>
-    <!-- Вызовы макроса leg для каждой ноги с передачей robot_name -->
-    <xacro:leg robot_name="$(arg robot_name)" name="FR" mirror="-1" mirror_dae="False" front_hind="1" front_hind_dae="True"/>
-    <xacro:leg robot_name="$(arg robot_name)" name="FL" mirror="1" mirror_dae="True" front_hind="1" front_hind_dae="True"/>
-    <xacro:leg robot_name="$(arg robot_name)" name="RR" mirror="-1" mirror_dae="False" front_hind="-1" front_hind_dae="False"/>
-    <xacro:leg robot_name="$(arg robot_name)" name="RL" mirror="1" mirror_dae="True" front_hind="-1" front_hind_dae="False"/>
-    <!-- Дополнительные сенсоры (закомментированы) -->
-    <!--
-    <xacro:depthCamera camID="1" name="${prefix}face">
+    <xacro:leg name="FR" mirror="-1" mirror_dae= "False" front_hind="1"  front_hind_dae="True"  />
+    <xacro:leg name="FL" mirror="1"  mirror_dae="True"   front_hind="1"  front_hind_dae="True"  />
+    <xacro:leg name="RR" mirror="-1" mirror_dae="False"  front_hind="-1" front_hind_dae="False" />
+    <xacro:leg name="RL" mirror="1"  mirror_dae="True"   front_hind="-1" front_hind_dae="False" />
+    <!-- <xacro:depthCamera camID="1" name="face">
         <origin rpy="${PI} 0 0" xyz="0.2785 0.0125 0.0167"/>
     </xacro:depthCamera>
-    <xacro:depthCamera camID="2" name="${prefix}chin">
+    <xacro:depthCamera camID="2" name="chin">
         <origin rpy="${PI} ${PI/2} 0" xyz="0.2522 0.0125 -0.0436"/>
     </xacro:depthCamera>
-    <xacro:depthCamera camID="3" name="${prefix}left">
+    <xacro:depthCamera camID="3" name="left">
         <origin rpy="${PI} 0.2618 ${PI/2}" xyz="-0.066 0.082 -0.0176"/>
     </xacro:depthCamera>
-    <xacro:depthCamera camID="4" name="${prefix}right">
+    <xacro:depthCamera camID="4" name="right">
         <origin rpy="${PI} 0.2618 ${-PI/2}" xyz="-0.041 -0.082 -0.0176"/>
     </xacro:depthCamera>
-    <xacro:depthCamera camID="5" name="${prefix}rearDown">
+    <xacro:depthCamera camID="5" name="rearDown">
         <origin rpy="${PI} ${PI/2} 0" xyz="-0.0825 0.0125 -0.04365"/>
     </xacro:depthCamera>
-    <joint name="${prefix}camera_laserscan_joint_left" type="fixed">
+    <joint name="camera_laserscan_joint_left" type="fixed">
         <origin rpy="0 0.2618 0" xyz="0 0 0"/>
-        <parent link="${prefix}camera_left"/>
-        <child link="${prefix}camera_laserscan_link_left"/>
+        <parent link="camera_left"/>
+        <child link="camera_laserscan_link_left"/>
     </joint>
-    <link name="${prefix}camera_laserscan_link_left">
+    <link name="camera_laserscan_link_left">
     </link>
-    <joint name="${prefix}camera_laserscan_joint_right" type="fixed">
+    <joint name="camera_laserscan_joint_right" type="fixed">
         <origin rpy="0 0.2618 0" xyz="0 0 0"/>
-        <parent link="${prefix}camera_right"/>
-        <child link="${prefix}camera_laserscan_link_right"/>
+        <parent link="camera_right"/>
+        <child link="camera_laserscan_link_right"/>
     </joint>
-    <link name="${prefix}camera_laserscan_link_right">
+    <link name="camera_laserscan_link_right">
     </link>
-    <xacro:ultraSound name="${prefix}left">
+    <xacro:ultraSound name="left">
         <origin rpy="0 0.2618 ${PI/2}" xyz="-0.0535  0.0826 0.00868"/>
     </xacro:ultraSound>
-    <xacro:ultraSound name="${prefix}right">
+    <xacro:ultraSound name="right">
         <origin rpy="0 0.2618 ${-PI/2}" xyz="-0.0535 -0.0826 0.00868"/>
     </xacro:ultraSound>
-    <xacro:ultraSound name="${prefix}face">
+    <xacro:ultraSound name="face">
         <origin rpy="0 0 0" xyz="0.2747 0.0 -0.0088"/>
-    </xacro:ultraSound>
-    -->
+    </xacro:ultraSound> -->
 </robot>

File: go1_description/xacro/transmission.xacro (robot description, xacro)
@@ -1,33 +1,33 @@
 <?xml version="1.0"?>
 <robot xmlns:xacro="http://www.ros.org/wiki/xacro">
-    <xacro:macro name="leg_transmission" params="robot_name name">
-        <transmission name="${robot_name}_${name}_hip_tran">
+    <xacro:macro name="leg_transmission" params="name">
+        <transmission name="${name}_hip_tran">
             <type>transmission_interface/SimpleTransmission</type>
-            <joint name="${robot_name}_${name}_hip_joint">
-                <hardwareInterface>hardware_interface/EffortJointInterface</hardwareInterface>
+            <joint name="${name}_hip_joint">
+            <hardwareInterface>hardware_interface/EffortJointInterface</hardwareInterface>
             </joint>
-            <actuator name="${robot_name}_${name}_hip_motor">
-                <hardwareInterface>hardware_interface/EffortJointInterface</hardwareInterface>
-                <mechanicalReduction>1</mechanicalReduction>
+            <actuator name="${name}_hip_motor">
+            <hardwareInterface>hardware_interface/EffortJointInterface</hardwareInterface>
+            <mechanicalReduction>1</mechanicalReduction>
             </actuator>
         </transmission>
-        <transmission name="${robot_name}_${name}_thigh_tran">
+        <transmission name="${name}_thigh_tran">
             <type>transmission_interface/SimpleTransmission</type>
-            <joint name="${robot_name}_${name}_thigh_joint">
-                <hardwareInterface>hardware_interface/EffortJointInterface</hardwareInterface>
+            <joint name="${name}_thigh_joint">
+            <hardwareInterface>hardware_interface/EffortJointInterface</hardwareInterface>
             </joint>
-            <actuator name="${robot_name}_${name}_thigh_motor">
-                <hardwareInterface>hardware_interface/EffortJointInterface</hardwareInterface>
-                <mechanicalReduction>1</mechanicalReduction>
+            <actuator name="${name}_thigh_motor">
+            <hardwareInterface>hardware_interface/EffortJointInterface</hardwareInterface>
+            <mechanicalReduction>1</mechanicalReduction>
             </actuator>
         </transmission>
-        <transmission name="${robot_name}_${name}_calf_tran">
+        <transmission name="${name}_calf_tran">
             <type>transmission_interface/SimpleTransmission</type>
-            <joint name="${robot_name}_${name}_calf_joint">
-                <hardwareInterface>hardware_interface/EffortJointInterface</hardwareInterface>
+            <joint name="${name}_calf_joint">
+            <hardwareInterface>hardware_interface/EffortJointInterface</hardwareInterface>
             </joint>
-            <actuator name="${robot_name}_${name}_calf_motor">
-                <hardwareInterface>hardware_interface/EffortJointInterface</hardwareInterface>
-                <mechanicalReduction>1</mechanicalReduction>
+            <actuator name="${name}_calf_motor">
+            <hardwareInterface>hardware_interface/EffortJointInterface</hardwareInterface>
+            <mechanicalReduction>1</mechanicalReduction>
             </actuator>
         </transmission>

Commit message: Added VV Files without Map

File: go1_description/xacro/gazebo.xacro (robot description, xacro)
@@ -144,5 +144,5 @@
             </sensor>
         </gazebo>
-        <gazebo reference="laser_frame">
+        <gazebo reference="laser_frame">                                                    <!-- LIDAR settings here -->
             <!--<material>Gazebo/Black</material>-->
             <sensor name="laser" type="gpu_lidar">

File: go1_description/xacro/robot.xacro (robot description, xacro)
@@ -14,4 +14,5 @@
     <xacro:include filename="$(find go1_description)/xacro/ultraSound.xacro"/>
     <!-- <xacro:include filename="$(find go1_description)/launch/stairs.urdf.xacro"/> -->
+    <xacro:include filename="$(find go1_description)/xacro/robosense_airy_lidar.xacro"/>     <!-- Included Robosense Airy Lidar xacro file -->
     <xacro:robot_gazebo_sensors robot_name="$(arg robot_name)"/>
     <joint name='laser_scan' type='fixed'>
@@ -144,3 +145,7 @@
         <origin rpy="0 0 0" xyz="0.2747 0.0 -0.0088"/>
     </xacro:ultraSound>
+     <xacro:Lidar_Robosense_Airy name="robosense_airy_lidar">                                       <!-- Added Robosense Airy Lidar macro call -->
+        <origin rpy="0 0 0" xyz="${lidar_x_offset} ${lidar_y_offset} ${lidar_z_offset}"/>
+        <parent>trunk</parent>
+    </xacro:Lidar_Robosense_Airy>
 </robot>
