Commit message: update

File: go2_description/xacro/gazebo.xacro (robot description, xacro)
@@ -117,5 +117,5 @@
                     </scan>
                     <range>
-                        <min>0.3</min>
+                        <min>0.05</min>
                         <max>12</max>
                     </range>

File: go2_description/xacro/laser.xacro (robot description, xacro)
@@ -26,5 +26,5 @@
         </inertial>
     </link>
-    <gazebo reference="front_laser">
+    <!-- <gazebo reference="front_laser">
         <sensor name="front_laser_sensor" type="ray">
             <always_on>true</always_on>
@@ -60,4 +60,4 @@
             </plugin>
         </sensor>
-    </gazebo>
+    </gazebo> -->
 </robot>

File: go2_description/xacro/robot.xacro (robot description, xacro)
@@ -157,4 +157,29 @@
     </link>
   -->
+    <joint name="camera_face_joint" type="fixed">
+        <parent link="base_link"/>
+        <child link="camera_face"/>
+        <origin xyz="0.33 0 0.0057" rpy="0 0 0"/>
+    </joint>
+    <link name="camera_face">
+        <inertial>
+            <mass value="0.001"/>
+            <origin rpy="0 0 0" xyz="0 0 0"/>
+            <inertia ixx="0.0001" ixy="0" ixz="0" iyy="0.0001" iyz="0" izz="0.0001"/>
+        </inertial>
+        <visual>
+            <origin rpy="0 0 0" xyz="0 0 0"/>
+            <geometry>
+                <box size="0.001 0.001 0.001"/>
+            </geometry>
+            <!-- <material name="red"/> -->
+        </visual>
+        <collision>
+            <origin rpy="0 0 0" xyz="0 0 0"/>
+            <geometry>
+                <box size="0.001 0.001 0.001"/>
+            </geometry>
+        </collision>
+    </link>
     <xacro:leg name="rf" mirror="-1" mirror_dae= "False" front_hind="1"  front_hind_dae="True"  />
     <xacro:leg name="lf" mirror="1"  mirror_dae="True"   front_hind="1"  front_hind_dae="True"  />

Commit message: Integrated V2C2 files, did work, now problem while loading plugin for gazebo.xacro

File: go2_description/xacro/gazebo.xacro (robot description, xacro)
@@ -102,8 +102,9 @@
             </sensor>
         </gazebo>
+        <!-- uncomment to add default lidar to the robot in gazebo -->
+        <!--
         <gazebo reference="laser_frame">
-            <!--<material>Gazebo/Black</material>-->
+            <material>Gazebo/Black</material>
             <sensor name="laser" type="gpu_lidar">
-            <!--<sensor name="laser" type="ray">-->
                 <pose> 0 0 0 0 0 0 </pose>
                 <visualize>true</visualize>
@@ -126,4 +127,5 @@
             </sensor>
         </gazebo>
+        -->
         <gazebo reference="camera_face">
             <!-- <material>Gazebo/Black</material> -->

File: go2_description/xacro/gazebo_lidar_robosense.xacro (robot description, xacro)
@@ -1,36 +1,36 @@
 <?xml version="1.0"?>
-<robot name="gazebo_ouster" xmlns:xacro="http://www.ros.org/wiki/xacro">
-  <xacro:macro name="gazebo_ouster" params="lidar_suffix
+<robot name="gazebo_lidar_robosense" xmlns:xacro="http://www.ros.org/wiki/xacro">
+  <xacro:macro name="gazebo_lidar_robosense" params="lidar_suffix
                                             calibration_parent:=sensor_kit_base_link
                                             robot_name">
-    <!-- Crate local variables -->
+    <!-- Create local variables -->
     <xacro:property name="M_PI" value="3.14159"/>
     <xacro:property name="lidar_name" value="lidar_${lidar_suffix}"/>
     <xacro:property name="parent" value="${calibration_parent}"/>
-   <!-- Include Sensor Calibration -->
-   <xacro:property name="calibration" value="${xacro.load_yaml('$(find go2_description)/xacro/sensor_kit_calibration.yaml')}"/>
+    <!-- Include Sensor Calibration -->
+    <xacro:property name="calibration" value="${xacro.load_yaml('$(find go2_description)/xacro/sensor_kit_calibration.yaml')}"/>
     <!-- Sensor Gazebo Lidar -->
     <!-- Note: Using dict.get('key', 'default-value') to use a default-value in case the key in the dict is missing -->
     <!-- Note2: Gazebo-lidar-plugin is only loaded if "simulate" in the yaml-configuration is set to true -->
-    <xacro:if value="${calibration[parent][lidar_name+'/os_sensor']['simulate']}">
+    <xacro:if value="${calibration[parent][lidar_name+'/airy_sensor']['simulate']}">
       <xacro:property name="lidar_range"
-                      value="${calibration[parent][lidar_name+'/os_sensor'].get('range', 50.0)}"/>
+                      value="${calibration[parent][lidar_name+'/airy_sensor'].get('range', 50.0)}"/>
       <xacro:property name="channels"
-                      value="${calibration[parent][lidar_name+'/os_sensor'].get('channels', 32)}"/>
+                      value="${calibration[parent][lidar_name+'/airy_sensor'].get('channels', 32)}"/>
       <xacro:property name="points_per_second"
-                      value="${calibration[parent][lidar_name+'/os_sensor'].get('points_per_second', 32000)}"/>
+                      value="${calibration[parent][lidar_name+'/airy_sensor'].get('points_per_second', 32000)}"/>
       <xacro:property name="upper_fov"
-                      value="${calibration[parent][lidar_name+'/os_sensor'].get('upper_fov', 22.5)}"/>
+                      value="${calibration[parent][lidar_name+'/airy_sensor'].get('upper_fov', 22.5)}"/>
       <xacro:property name="lower_fov"
-                      value="${calibration[parent][lidar_name+'/os_sensor'].get('lower_fov', -22.5)}"/>
+                      value="${calibration[parent][lidar_name+'/airy_sensor'].get('lower_fov', -22.5)}"/>
       <xacro:property name="frequency"
-                      value="${calibration[parent][lidar_name+'/os_sensor'].get('rotation_frequency', 10)}"/>
+                      value="${calibration[parent][lidar_name+'/airy_sensor'].get('rotation_frequency', 10)}"/>
       <xacro:property name="noise_stddev"
-                      value="${calibration[parent][lidar_name+'/os_sensor'].get('noise_stddev', 0.0)}"/>
+                      value="${calibration[parent][lidar_name+'/airy_sensor'].get('noise_stddev', 0.0)}"/>
       <xacro:property name="gz_topic"
-                      value="${calibration[parent][lidar_name+'/os_sensor'].get('topic', '/sensing/lidar/'+lidar_suffix)}"/>
+                      value="${calibration[parent][lidar_name+'/airy_sensor'].get('topic', '/sensing/lidar/'+lidar_suffix)}"/>
       <gazebo reference="laser_frame">
-      <!-- <gazebo reference="${lidar_name}/os_lidar"> -->
-        <sensor type="gpu_lidar" name="${lidar_name}/os_lidar">
+      <!--<gazebo reference="${lidar_name}/robosense_airy_lidar"> -->
+        <sensor type="gpu_lidar" name="${lidar_name}/robosense_airy_lidar">
           <pose>0 0 0 0 0 0</pose>
           <visualize>true</visualize>

File: go2_description/xacro/robot.xacro (robot description, xacro)
@@ -6,7 +6,13 @@
     <xacro:include filename="$(find go2_description)/xacro/leg.xacro"/>
     <!-- <xacro:include filename="$(find go2_description)/xacro/stairs.xacro"/> -->
+    <!-- <xacro:include filename="$(find go2_description)/launch/stairs.urdf.xacro"/> -->
     <xacro:include filename="$(find go2_description)/xacro/gazebo.xacro"/>
-    <!-- <xacro:include filename="$(find go2_description)/launch/stairs.urdf.xacro"/> -->
     <xacro:robot_gazebo_sensors robot_name="$(arg robot_name)"/>
+    <xacro:include filename="$(find go2_description)/xacro/gazebo_ouster.xacro"/>
+    <xacro:gazebo_ouster lidar_suffix="top" calibration_parent="sensor_kit_base_link" robot_name="$(arg robot_name)"/>
+    <!--
+    <xacro:include filename="$(find go2_description)/xacro/gazebo_lidar_robosense.xacro"/>
+    <xacro:gazebo_lidar_robosense lidar_suffix="top" calibration_parent="sensor_kit_base_link" robot_name="$(arg robot_name)"/>
+    -->
     <!-- <xacro:stairs stairs="15" xpos="0" ypos="0" zpos="0" /> -->
     <!-- Rotor related joint and link is only for demonstrate location. -->
@@ -72,4 +78,6 @@
             <geometry>
                 <cylinder length="0.01" radius="0.018" />
+                <!-- <mesh filename="file://$(find go2_description)/meshes/ouster_os2.dae" scale="0.001 0.001 0.001"/> -->   <!-- still a little to big and not rotated correctly but works-->
+                <!-- <mesh filename="file://$(find go2_description)/meshes/robosense_airy.dae" scale="1 1 1"/> -->  <!-- for some reason this file does not work -->
             </geometry>
             <!-- <material name="red"/> -->
